File: eggbot-spherebot-polargraph-controller.kicad_pcb (KiCad board)
At the start: 2 copper layers, 83.8 x 43.2 mm, 17 parts, among them CON1 12V DC, P1 Stepper1, P2 Stepper2, P3 Endstop1 (A1), P4 Endstop2 (A2), P5 Servo (A0), P6 EXT PWR, P7 SD Card (SPI), U1 Arduino_Nano, U2 STEPSTICK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

Commit message: Updated readme and licence details
Parts:
- P7: value SD Card (SPI) -> SPI
Other:
- board text added: "-"
- board text added: "©Mark Benson 2016 CC BY-NC-SA"
- board text removed: "©Mark Benson 2015 CCNC"
Changed lines of the file:
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@@
 (kicad_pcb (version 4) (host pcbnew 4.0.2-stable)
   (general
-    (links 0)
+    (links 57)
     (no_connects 0)
-    (area 115.431474 63.4545 206.610046 108.84626)
+    (area 118.059999 64.719999 201.980001 108.000001)
     (thickness 1.6)
-    (drawings 8)
+    (drawings 10)
     (tracks 192)
     (zones 0)
@@
       (effects (font (size 1 1) (thickness 0.15)))
     )
-    (fp_text value "SD Card (SPI)" (at 2.794 7.366 450) (layer F.SilkS)
+    (fp_text value SPI (at 2.794 7.366 270) (layer F.SilkS)
       (effects (font (size 1 1) (thickness 0.15)))
     )
@@
     )
   )
+  (gr_text - (at 120.65 81.534) (layer F.SilkS)
+    (effects (font (size 1.5 1.5) (thickness 0.3)))
+  )
+  (gr_text - (at 145.796 81.534) (layer F.SilkS)
+    (effects (font (size 1.5 1.5) (thickness 0.3)))
+  )
   (gr_text github.com/markjb (at 154.94 91.44) (layer F.SilkS)
     (effects (font (size 1 1) (thickness 0.2)))
@@
     (effects (font (size 1 1) (thickness 0.2)))
   )
-  (gr_text "Arduino Nano dual stepper board v2.2" (at 137.795 89.535) (layer F.SilkS)
+  (gr_text "Arduino Nano dual stepper board v2.2" (at 133.858 89.662) (layer F.SilkS)
     (effects (font (size 0.8 0.8) (thickness 0.2)))
   )
-  (gr_text "©Mark Benson 2015 CCNC" (at 161.29 89.535) (layer F.SilkS)
+  (gr_text "©Mark Benson 2016 CC BY-NC-SA" (at 160.528 89.662) (layer F.SilkS)
     (effects (font (size 1 1) (thickness 0.2)))
   )
